File: sindo.kicad_pcb (KiCad board)
At the start: 2 copper layers, 153 parts, among them J1 Conn_02x06_Top_Bottom, J2 Conn_02x06_Top_Bottom, U1 ESP32DEVKITV1

Commit message: Started with the first half layout
Parts:
- D1, D10, D11, D12, D13, D14, D15, D16, D17, D18, D19, D2, D20, D21, D22, D23, D24, D25, D26, D27, D28, D29, D3, D30, D31, D32, D33, D34, D35, D36, D37, D38, D39, D4, D40, D41, D42, D43, D44, D45, D46, D47, D48, D49, D5, D50, D51, D52, D53, D54, D55, D56, D57, D58, D59, D6, D60, D61, D62, D63, D64, D65, D66, D67, D68, D69, D7, D70, D71, D72, D8, D9: footprint Diode_THT:D_DO-35_SOD27_P3.81mm_Vertical_AnodeUp -> Diode_THT:D_DO-35_SOD27_P7.62mm_Horizontal
- moved MX4 413.4 mm to (-196.8, -4.76)
- moved D7 408.8 mm to (-169.4, -59.4), turned to 90 degrees
- moved MX5 401.9 mm to (-196.8, 14.3)
- moved MX7 384.4 mm to (-177.8, -61.9)
- moved MX8 373.7 mm to (-177.8, -42.9)
- moved D13 364.7 mm to (-150.4, -67.3), turned to 90 degrees
- moved MX9 359.4 mm to (-177.8, -23.8)
- moved D19 345.1 mm to (-131.3, -70.5), turned to 90 degrees
- moved MX14 343.7 mm to (-158.8, -50.8)
- moved MX10 340.7 mm to (-177.8, -4.76)
- moved D31 329.8 mm to (-93.2, -61.0), turned to 90 degrees
- moved MX15 325.3 mm to (-158.8, -31.8)
- moved MX13 324.3 mm to (-158.8, -69.8)
- moved MX11 322.2 mm to (-177.8, 14.3)
- moved MX28 317.5 mm to (-120.7, -12.7)
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
Commit message: Almost done with layout
Parts:
- moved D2 404.7 mm to (-188.5, -38.7), turned to 90 degrees
- moved D4 400.3 mm to (-188.5, -0.65), turned to 90 degrees
- moved D3 393.9 mm to (-188.5, -19.7), turned to 90 degrees
- moved D9 390.0 mm to (-169.5, -21.3), turned to 90 degrees
- moved D5 383.9 mm to (-188.5, 18.4), turned to 90 degrees
- moved D17 374.6 mm to (-150.4, 8.89), turned to 90 degrees
- moved D16 370.0 mm to (-150.4, -10.2), turned to 90 degrees
- moved D11 368.5 mm to (-169.5, 16.8), turned to 90 degrees
- moved D20 366.0 mm to (-131.4, -51.4), turned to 90 degrees
- moved D15 364.5 mm to (-150.4, -29.2), turned to 90 degrees
- moved D14 363.9 mm to (-150.4, -48.3), turned to 90 degrees
- moved D22 362.0 mm to (-131.4, -13.3), turned to 90 degrees
- moved D23 360.1 mm to (-131.4, 5.70), turned to 90 degrees
- moved D8 343.1 mm to (-169.4, -40.3), turned to 90 degrees
- moved D29 340.8 mm to (-112.3, 8.89), turned to 90 degrees
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
Commit message: Done with the basic layout
Parts:
- moved D68 232.6 mm to (141.7, -38.7), turned to 90 degrees
- moved D62 231.2 mm to (122.7, -40.3), turned to 90 degrees
- moved D69 219.8 mm to (141.7, -19.7), turned to 90 degrees
- moved D56 213.2 mm to (103.6, -48.3), turned to 90 degrees
- moved D57 208.6 mm to (103.6, -29.2), turned to 90 degrees
- moved D72 205.8 mm to (27.4, -56.2), turned to 90 degrees
- moved D63 203.4 mm to (122.6, -21.3), turned to 90 degrees
- moved D70 198.6 mm to (141.7, -0.64), turned to 90 degrees
- moved D58 191.8 mm to (103.6, -10.2), turned to 90 degrees
- moved D71 191.6 mm to (141.7, 18.4), turned to 90 degrees
- moved D64 185.4 mm to (122.7, -2.22), turned to 90 degrees
- moved D65 179.0 mm to (122.6, 16.9), turned to 90 degrees
- moved D66 171.5 mm to (27.4, -37.1), turned to 90 degrees
- moved D59 162.8 mm to (103.6, 8.89), turned to 90 degrees
- moved D60 155.5 mm to (27.4, -18.1), turned to 90 degrees
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
Commit message: Using a better header footprint.
Parts:
- J1, J2: value Conn_02x06_Top_Bottom -> Conn_02x06_Odd_Even
- moved U1 418.6 mm to (238.1, 115.9), turned to 180 degrees
- moved J2 405.0 mm to (341.3, 132.6)
- moved D1 391.9 mm to (136.9, 160.5)
- moved D10 391.9 mm to (156.0, 216.1)
- moved D11 391.9 mm to (156.0, 235.1)
- moved D12 391.9 mm to (251.2, 181.1)
- moved D13 391.9 mm to (175.1, 150.9)
- moved D14 391.9 mm to (175.1, 170.0)
- moved D15 391.9 mm to (175.0, 189.1)
- moved D16 391.9 mm to (175.0, 208.1)
- moved D17 391.9 mm to (175.0, 227.2)
- moved D18 391.9 mm to (251.2, 200.2)
- moved D19 391.9 mm to (194.2, 147.8)
- moved D2 391.9 mm to (136.9, 179.5)
- moved D20 391.9 mm to (194.1, 166.8)
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Connections:
- J1 pad 10: COL9 -> COL10
- J1 pad 11: COL10 -> ROW5
- J1 pad 2: ROW1 -> COL6
- J1 pad 3: ROW2 -> ROW1
- J1 pad 4: ROW3 -> COL7
- J1 pad 5: ROW4 -> ROW2
- J1 pad 6: ROW5 -> COL8
- J1 pad 7: COL6 -> ROW3
- J1 pad 8: COL7 -> COL9
- J1 pad 9: COL8 -> ROW4
- J2 pad 10: C9 -> C10
- J2 pad 11: C10 -> R5
- J2 pad 2: R1 -> C6
- J2 pad 3: R2 -> R1
- J2 pad 4: R3 -> C7
- J2 pad 5: R4 -> R2
- J2 pad 6: R5 -> C8
- J2 pad 7: C6 -> R3
- J2 pad 8: C7 -> C9
- J2 pad 9: C8 -> R4

Commit message: Reworked the layout for a single layer
Parts:
- moved U1 171.0 mm to (75.2, 64.0)
- moved MX37 128.7 mm to (249.8, 94.4)
- moved MX38 128.7 mm to (249.8, 113.5)
- moved MX39 128.7 mm to (249.8, 132.5)
- moved MX40 128.7 mm to (249.8, 151.6)
- moved D37 128.7 mm to (258.2, 97.0)
- moved D38 128.7 mm to (258.2, 116.0)
- moved D40 128.7 mm to (258.2, 154.1)
- moved D42 128.7 mm to (245.5, 197.0)
- moved D43 128.7 mm to (277.2, 90.6)
- moved D44 128.7 mm to (277.3, 109.7)
- moved D45 128.7 mm to (277.2, 128.7)
- moved D46 128.7 mm to (277.2, 147.8)
- moved D49 128.7 mm to (296.3, 87.4)
- moved D50 128.7 mm to (296.3, 106.5)
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Connections:
- J1 pad 1: ROW0 -> ROW5
- J1 pad 10: COL10 -> COL7
- J1 pad 11: ROW5 -> ROW0
- J1 pad 12: COL11 -> COL6
- J1 pad 2: COL6 -> COL11
- J1 pad 3: ROW1 -> ROW4
- J1 pad 4: COL7 -> COL10
- J1 pad 5: ROW2 -> ROW3
- J1 pad 6: COL8 -> COL9
- J1 pad 7: ROW3 -> ROW2
- J1 pad 8: COL9 -> COL8
- J1 pad 9: ROW4 -> ROW1
- J2 pad 1: R0 -> R5
- J2 pad 10: C10 -> C7
- J2 pad 11: R5 -> R0
- J2 pad 12: C11 -> C6
- J2 pad 2: C6 -> C11
- J2 pad 3: R1 -> R4
- J2 pad 4: C7 -> C10
- J2 pad 5: R2 -> R3
- J2 pad 6: C8 -> C9
- J2 pad 7: R3 -> R2
- J2 pad 8: C9 -> C8
- J2 pad 9: R4 -> R1
- U1 pad D32: ROW4 -> ROW1
- U1 pad D33: ROW5 -> ROW0
- U1 pad D34: ROW2 -> ROW3
- U1 pad D35: ROW3 -> ROW2
- U1 pad D36: ROW0 -> ROW5
- U1 pad D39: ROW1 -> ROW4
Routing:
- net ROW5: track 0.00 -> 543.2 mm
- net COL0: track 0.00 -> 473.6 mm, vias 0 -> 12
- net ROW4: track 0.00 -> 413.6 mm
- net COL1: track 0.00 -> 413.5 mm, vias 0 -> 13
- net ROW3: track 0.00 -> 387.0 mm
- net COL2: track 0.00 -> 376.3 mm, vias 0 -> 13
- net ROW2: track 0.00 -> 366.1 mm
- net ROW1: track 0.00 -> 344.3 mm
- net R3: track 0.00 -> 268.6 mm, vias 0 -> 2
- net R4: track 0.00 -> 263.7 mm, vias 0 -> 2
- net R2: track 0.00 -> 242.2 mm
- net COL5: track 0.00 -> 237.8 mm, vias 0 -> 10
- net COL3: track 0.00 -> 232.8 mm, vias 0 -> 11
- net ROW0: track 0.00 -> 229.4 mm
- net R1: track 0.00 -> 221.1 mm
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Other:
- net class Default: trace_width 0.25 -> 0.9; via_dia 0.8 -> 2

Commit message: Finished the Sindo PCB V1
Parts:
- moved MX37 30.6 mm to (268.8, 70.4)
- moved MX38 30.6 mm to (268.8, 89.5)
- moved MX40 30.6 mm to (268.8, 127.6)
- moved MX42 30.6 mm to (256.1, 170.4)
- moved D39 30.6 mm to (277.2, 111.1)
- moved D63 30.6 mm to (353.4, 112.7)
- moved MX46 30.6 mm to (287.9, 121.2)
- moved MX58 30.6 mm to (326.0, 121.2)
- moved MX60 30.6 mm to (249.8, 113.3)
- moved J2 30.6 mm to (245.8, 57.8)
- moved MX49 30.6 mm to (306.9, 60.9)
- moved MX39 30.6 mm to (268.8, 108.5)
- moved D37 30.6 mm to (277.2, 73.0)
- moved D38 30.6 mm to (277.2, 92.0)
- moved D40 30.6 mm to (277.2, 130.1)
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Routing:
- net R5: track 0.00 -> 307.3 mm, vias 0 -> 6
- net C9: track 88.2 -> 319.9 mm, vias 0 -> 13
- net C8: track 63.0 -> 274.9 mm, vias 0 -> 10
- net C10: track 118.0 -> 297.3 mm, vias 0 -> 13
- net C6: track 17.6 -> 159.6 mm, vias 0 -> 8
- net C7: track 37.3 -> 156.9 mm, vias 0 -> 10
- net C11: track 145.1 -> 262.2 mm, vias 0 -> 11
- net GND: track 50.2 -> 61.0 mm, vias 0 -> 2
- net Net-(D14-Pad2): track 0.00 -> 5.83 mm
- net ROW5: track 543.2 -> 538.0 mm
- net ROW3: track 387.0 -> 384.1 mm, vias 0 -> 2
- net ROW2: track 366.1 -> 363.2 mm, vias 0 -> 2
- net ROW4: track 413.6 -> 410.8 mm, vias 0 -> 2
- net ROW1: track 344.3 -> 342.0 mm, vias 0 -> 2
- net ROW0: track 229.4 -> 231.1 mm, vias 0 -> 2
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Other:
- board outline added: 350 x 190 mm

Commit message: Added more realistic footprints for the headers and resistors
Parts:
- J1, J2: footprint Connector_PinHeader_1.27mm:PinHeader_2x06_P1.27mm_Vertical -> Connector_PinHeader_2.54mm:PinHeader_2x06_P2.54mm_Vertical
- R1, R2, R3, R4, R5, R6: footprint Resistor_THT:R_Axial_DIN0207_L6.3mm_D2.5mm_P5.08mm_Vertical -> Resistor_THT:R_Axial_DIN0411_L9.9mm_D3.6mm_P7.62mm_Vertical
- moved J2 6.19 mm to (239.7, 58.3)
- moved R4 3.66 mm to (64.1, 31.3)
- moved R6 3.66 mm to (58.1, 31.3)
- moved R1 3.66 mm to (73.1, 31.3)
- moved R5 3.66 mm to (61.1, 31.3)
- moved R2 3.66 mm to (70.1, 31.3)
- moved R3 3.66 mm to (67.1, 31.3)
- moved J1 1.07 mm to (177.0, 58.0)
Routing:
- net C11: track 262.2 -> 274.6 mm
- net R4: track 263.7 -> 257.3 mm
- net R5: track 307.3 -> 300.9 mm
- net C8: track 274.9 -> 280.8 mm
- net R3: track 268.6 -> 263.1 mm
- net ROW0: track 231.1 -> 236.4 mm
- net C9: track 319.9 -> 314.7 mm, vias 13 -> 14
- net R2: track 242.2 -> 237.4 mm
- net ROW1: track 342.0 -> 346.3 mm
- net R1: track 221.1 -> 216.8 mm
- net C7: track 156.9 -> 161.2 mm
- net COL6: track 108.5 -> 112.3 mm
- net ROW2: track 363.2 -> 366.7 mm
- net R0: track 201.1 -> 197.7 mm
- net COL7: track 110.0 -> 112.8 mm
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